File: BLDC_SensorlessWithLM339/BLDC_SensorlessWithLM339.sch (KiCad schematic (older format))
At the start: 48 parts, among them J1 Conn_01x04_Female, J2 Conn_01x07_Female, J3 Screw_Terminal_01x02, J4 Screw_Terminal_01x03, Q1 50N06, Q2 50N06, Q3 50N06, Q4 50N06, Q5 50N06, Q6 50N06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

Commit message: Version 0.3
I ordered the PCB. I will test it when it arrives.
Parts:
- added C1: 10u, Capacitor_THT:CP_Radial_D5.0mm_P2.50mm, symbol Device:CP1_Small
- added D4, D5, D6, D7, D8, D9: 1N4148, Diode_THT:D_DO-35_SOD27_P7.62mm_Horizontal, symbol Diode:1N4148
- C2: renamed from C1; footprint Capacitor_THT:CP_Radial_D10.0mm_P5.00mm -> Capacitor_THT:CP_Radial_D5.0mm_P2.50mm; W2B (none) -> https://ozdisan.com/pasif-komponentler/kondansatorler/alumi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
- C3: renamed from C2; footprint Capacitor_THT:CP_Radial_D10.0mm_P5.00mm -> Capacitor_THT:CP_Radial_D5.0mm_P2.50mm; W2B (none) -> https://ozdisan.com/pasif-komponentler/kondansatorler/alumi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
- C4: renamed from C3; footprint Capacitor_THT:CP_Radial_D10.0mm_P5.00mm -> Capacitor_THT:CP_Radial_D5.0mm_P2.50mm; W2B (none) -> https://ozdisan.com/pasif-komponentler/kondansatorler/alumi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
- C5: renamed from C4; footprint Capacitor_THT:CP_Radial_D12.5mm_P5.00mm -> Capacitor_THT:CP_Radial_D5.0mm_P2.50mm; W2B (none) -> https://ozdisan.com/pasif-komponentler/kondansatorler/alumi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
- C6: renamed from C5; footprint Capacitor_THT:CP_Radial_D12.5mm_P5.00mm -> Capacitor_THT:CP_Radial_D5.0mm_P2.50mm; W2B (none) -> https://ozdisan.com/pasif-komponentler/kondansatorler/alumi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
- C7: renamed from C6; footprint Capacitor_THT:CP_Radial_D12.5mm_P5.00mm -> Capacitor_THT:CP_Radial_D5.0mm_P2.50mm; W2B (none) -> https://ozdisan.com/pasif-komponentler/kondansatorler/alumi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
- R10, R13, R14, R15, R8, R9: value 220 -> 10k
- R11, R12, R4, R5, R6, R7: value 10_2W -> 10_1W
- R16, R17, R18, R22, R23, R24: footprint Resistor_SMD:R_1206_3216Metric_Pad1.30x1.75mm_HandSolder -> Resistor_SMD:R_0805_2012Metric_Pad1.20x1.40mm_HandSolder
- renumbered C7 to C8, J2 to J1, J1 to J2
Connections:
- net +3V3: now also C1.1
- net GND: now also C1.2
- net at R12.1, U1.5 (LO): now also D8.1 (K)
- net at R11.1, U1.7 (HO): now also D9.1 (K)
- net at R6.1, U2.5 (LO): now also D6.1 (K)
- net at R5.1, U2.7 (HO): now also D5.1 (K)
- net at R7.1, U3.5 (LO): now also D7.1 (K)
- net at R4.1, U3.7 (HO): now also D4.1 (K)
- net at Q3.2 (G), R11.2, R14.1: now also D9.2 (A)
- net at Q4.2 (G), R12.2, R15.1: now also D8.2 (A)
- net at Q1.2 (G), R10.1, R5.2: now also D5.2 (A)
- net at Q2.2 (G), R6.2, R8.1: now also D6.2 (A)
- net at Q5.2 (G), R4.2, R9.1: now also D4.2 (A)
- net at Q6.2 (G), R13.1, R7.2: now also D7.2 (A)
